File: Sweep-half-swept/half-swept.kicad_pcb (KiCad board)
At the start: 2 copper layers, 108.6 x 86.9 mm, 26 parts, among them J2 AudioJack4dpb, SW10 SW_Push, SW11 SW_Push, SW12 SW_Push, SW14 SW_Push, SW15 SW_Push, SW16 SW_Push, SW17 SW_Push, SW18 SW_Push, SW2 SW_Push, SW2 SW_SPDT, SW20 SW_Push, SW21 SW_Push, SW3 SW_Push, SW4 SW_Push, SW5 SW_Push, SW6 SW_Push, SW8 SW_Push, SW9 SW_Push, U1 ProMicro-kbd

Commit message: remove pointless trace
Routing:
- net vcc: track 58.5 -> 53.0 mm

Commit message: Refactor repository and fix breakaway tabs
Parts:
- moved SW21 7.18 mm to (90.8, 87.0)
- moved SW15 7.18 mm to (45.1, 68.1)
- moved SW9 7.18 mm to (45.1, 51.1)
- moved Bat+r1 7.18 mm to (126.5, 46.0)
- moved BatGND1 7.18 mm to (111.3, 46.0)
- moved G*** 7.18 mm to (64.0, 82.0)
- moved J2 7.18 mm to (123.7, 82.8)
- moved REF** 7.18 mm to (72.6, 43.0)
- moved RSW1 7.18 mm to (79.2, 22.1)
- moved SW10 7.18 mm to (63.1, 44.2)
- moved SW11 7.18 mm to (81.1, 49.5)
- moved SW12 7.18 mm to (99.1, 52.1)
- moved SW14 7.18 mm to (27.1, 80.1)
- moved SW16 7.18 mm to (63.1, 61.2)
- moved SW17 7.18 mm to (81.1, 66.5)
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
Commit message: Update silk and edge cuts
Parts:
- POWER SW: renamed from SW_POWERR1
- renumbered Bat+r1 to B+, BatGND1 to B-
Other:
- board size 108.6 x 86.9 mm -> 109 x 86.9 mm
- board text added: "B+"
- board text added: "B-"
- board text added: "POWER SW"
- board text added: "TRRS"
