File: [PRE-RELEASE] Sweep Bling MX/bottom-plate/sweep-bling-mx__bottom.kicad_pcb (KiCad board)
At the start: 2 copper layers, 113.5 x 95.2 mm, 8 parts

Commit message: Update readmes and gerbers
Parts:
- mouse-bite-5mm-slot: value VAL** -> Mouse Bite 2
- mouse-bite-5mm-slot: value VAL** -> Mouse Bite 3
- mouse-bite-5mm-slot: value VAL** -> Mouse Bite 4
- mouse-bite-5mm-slot: value VAL** -> Mouse Bite 1
Changed lines of the file:
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@@
     (47 F.CrtYd user)
     (48 B.Fab user)
-    (49 F.Fab user hide)
+    (49 F.Fab user)
   )
   (setup
@@
       (effects (font (size 1 1) (thickness 0.2)))
     )
-    (fp_text value VAL** (at 0 0) (layer F.SilkS) hide
+    (fp_text value "Mouse Bite 2" (at 0 0) (layer F.SilkS) hide
       (effects (font (size 1 1) (thickness 0.2)))
     )
@@
       (effects (font (size 1 1) (thickness 0.2)))
     )
-    (fp_text value VAL** (at 0 0 90) (layer F.SilkS) hide
+    (fp_text value "Mouse Bite 3" (at 0 0 90) (layer F.SilkS) hide
       (effects (font (size 1 1) (thickness 0.2)))
     )
@@
       (effects (font (size 1 1) (thickness 0.2)))
     )
-    (fp_text value VAL** (at 0 0) (layer F.SilkS) hide
+    (fp_text value "Mouse Bite 4" (at 0 0) (layer F.SilkS) hide
       (effects (font (size 1 1) (thickness 0.2)))
     )
@@
       (effects (font (size 1 1) (thickness 0.2)))
     )
-    (fp_text value VAL** (at 0 0 90) (layer F.SilkS) hide
+    (fp_text value "Mouse Bite 1" (at 0 0 90) (layer F.SilkS) hide
       (effects (font (size 1 1) (thickness 0.2)))
     )
