File: [PRE-RELEASE] Sweep Bling MX/switch-plate/sweep-bling-mx__plate.kicad_pcb (KiCad board)
At the start: 2 copper layers, 111.6 x 95.2 mm, 26 parts, among them SW10 SW_Push, SW11 SW_Push, SW12 SW_Push, SW14 SW_Push, SW15 SW_Push, SW16 SW_Push, SW17 SW_Push, SW18 SW_Push, SW2 SW_Push, SW20 SW_Push, SW21 SW_Push, SW3 SW_Push, SW4 SW_Push, SW5 SW_Push, SW6 SW_Push, SW8 SW_Push, SW9 SW_Push

Commit message: Update readmes and gerbers
Other:
- board text added: "v0.1α"
Changed lines of the file:
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@@
   (general
     (thickness 1.6)
-    (drawings 17)
+    (drawings 18)
     (tracks 0)
     (zones 0)
@@
       (xy 1.415662 8.375391)) (layer B.Mask) (width 0.01))
   )
+  (gr_text v0.1α (at 44.6405 65.8495) (layer F.SilkS)
+    (effects (font (size 1 1) (thickness 0.15)))
+  )
   (gr_arc (start 145.9484 123.520494) (end 146.837399 124.155493) (angle -125.5376778) (layer Edge.Cuts) (width 0.05))
