File: Sweep High M/sweep-high.kicad_pcb (KiCad board)
At the start: 2 copper layers, 113.5 x 95.2 mm, 25 parts, among them J2 AudioJack4dpb, SW10 SW_Push, SW11 SW_Push, SW12 SW_Push, SW14 SW_Push, SW15 SW_Push, SW16 SW_Push, SW17 SW_Push, SW18 SW_Push, SW2 SW_Push, SW2 SW_SPDT, SW20 SW_Push, SW21 SW_Push, SW3 SW_Push, SW4 SW_Push, SW5 SW_Push, SW6 SW_Push, SW8 SW_Push, SW9 SW_Push, U1 ProMicro-kbd

Commit message: Fix DRC on sweep high m
Routing:
- net Switch7: track 108.2 -> 107.5 mm
Changed lines of the file:
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@@
   (segment (start 139.049239 117.400761) (end 140.8 119.151522) (width 0.25) (layer "B.Cu") (net 2))
   (segment (start 140.73 121.43) (end 140.75 121.45) (width 0.25) (layer "F.Cu") (net 3))
-  (segment (start 139.97 121.014) (end 139.99 121.034) (width 0.25) (layer "F.Cu") (net 3))
   (segment (start 140.73 116.82) (end 140.73 121.43) (width 0.25) (layer "F.Cu") (net 3))
   (segment (start 139.97 96.0434) (end 147.7054 88.308) (width 0.25) (layer "B.Cu") (net 3))
@@
   (segment (start 60.19 80.264) (end 60.19 81.534) (width 0.25) (layer "F.Cu") (net 11))
   (segment (start 129.50144 95.486912) (end 129.50144 99.712842) (width 0.25) (layer "F.Cu") (net 11))
+  (segment (start 112.208101 82.962727) (end 116.728577 87.483203) (width 0.25) (layer "F.Cu") (net 11))
   (segment (start 110.032653 80.042859) (end 110.107141 80.042859) (width 0.25) (layer "F.Cu") (net 11))
   (segment (start 133.89198 108.37406) (end 133.63804 108.628) (width 0.25) (layer "F.Cu") (net 11))
@@
   (segment (start 119.709466 91.202313) (end 125.197687 91.202313) (width 0.25) (layer "F.Cu") (net 11))
   (segment (start 125.207264 91.192736) (end 129.50144 95.486912) (width 0.25) (layer "F.Cu") (net 11))
-  (segment (start 112.208101 82.962727) (end 116.622687 87.377313) (width 0.25) (layer "F.Cu") (net 11))
   (segment (start 104.347688 72.402312) (end 104.35 72.4) (width 0.25) (layer "F.Cu") (net 11))
-  (segment (start 116.097687 86.852313) (end 116.728577 87.483203) (width 0.25) (layer "F.Cu") (net 11))
   (segment (start 129.4459 99.768382) (end 129.4459 100.200526) (width 0.25) (layer "F.Cu") (net 11))
   (segment (start 133.63804 108.628) (end 132.4854 108.628) (width 0.25) (layer "F.Cu") (net 11))
@@
   (segment (start 144.184831 106.088) (end 147.7054 106.088) (width 0.25) (layer "F.Cu") (net 19))
   (segment (start 110.133349 118.723696) (end 108.249223 120.607822) (width 0.25) (layer "F.Cu") (net 20))
-  (segment (start 139.55 119.95) (end 139.1 120.4) (width 0.25) (layer "F.Cu") (net 20))
   (segment (start 139.05 120.4) (end 139.05 123.164282) (width 0.25) (layer "F.Cu") (net 20))
   (segment (start 140.094511 114.794511) (end 139.1 115.789022) (width 0.25) (layer "F.Cu") (net 20))
   (segment (start 110.133349 119.419795) (end 110.133349 118.723696) (width 0.25) (layer "F.Cu") (net 20))
   (segment (start 108.249223 120.607822) (end 108.249223 120.848448) (width 0.25) (layer "F.Cu") (net 20))
-  (segment (start 139.1 120.4) (end 139.05 120.4) (width 0.25) (layer "F.Cu") (net 20))
+  (segment (start 139.55 119.95) (end 139.5 119.95) (width 0.25) (layer "F.Cu") (net 20))
   (segment (start 115.001714 124.28816) (end 110.133349 119.419795) (width 0.25) (layer "F.Cu") (net 20))
   (segment (start 139.1 115.789022) (end 139.1 117.657521) (width 0.25) (layer "F.Cu") (net 20))
   (segment (start 137.926122 124.28816) (end 115.001714 124.28816) (width 0.25) (layer "F.Cu") (net 20))
+  (segment (start 139.5 119.95) (end 139.05 120.4) (width 0.25) (layer "F.Cu") (net 20))
   (segment (start 147.7054 111.168) (end 144.078889 114.794511) (width 0.25) (layer "F.Cu") (net 20))
   (segment (start 139.1 117.657521) (end 139.05 117.707521) (width 0.25) (layer "F.Cu") (net 20))
@@
   (segment (start 141.352 86.065) (end 141.352 85.89) (width 0.25) (layer "B.Cu") (net 23))
   (segment (start 143.506 83.736) (end 146.19 83.736) (width 0.25) (layer "B.Cu") (net 23))
-  (zone (net 1) (net_name "gnd") (layer "F.Cu") (hatch edge 0.508)
+  (zone (net 1) (net_name "gnd") (layers F&B.Cu) (hatch edge 0.508)
     (connect_pads (clearance 0.508))
     (min_thickness 0.254) (filled_areas_thickness no)
-    (fill yes (thermal_gap 0.508) (thermal_bridge_width 0.508))
+    (fill yes (thermal_gap 0.508) (thermal_bridge_width 0.508) (island_removal_mode 1) (island_area_min 0))
     (polygon
       (pts
-        (xy 268.891231 40.704121)
-        (xy 268.891231 148.146121)
-        (xy 248.571231 148.400121)
-        (xy 22.003231 145.606121)
-        (xy 22.765231 40.450121)
+        (xy 151.476154 47.910806)
+        (xy 151.841623 146.745334)
+        (xy 30.791298 146.150384)
+        (xy 30.7848 47.0916)
       )
     )
-  )
-  (zone (net 1) (net_name "gnd") (layer "B.Cu") (hatch edge 0.508)
-    (connect_pads (clearance 0.508))
-    (min_thickness 0.254) (filled_areas_thickness no)
-    (fill yes (thermal_gap 0.508) (thermal_bridge_width 0.508))
-    (polygon
-      (pts
-        (xy 270.609675 40.937)
-        (xy 270.609675 146.861119)
-        (xy 250.289675 147.115119)
-        (xy 23.721675 144.321119)
-        (xy 24.483675 40.683)
-      )
-    )
