File: Sweep Compact LOW/ferris-sweep-compact.kicad_pcb (KiCad board)
At the start: 2 copper layers, 107.2 x 86.9 mm, 21 parts, among them J1 MJ-4PP-9, SW10 SW_PUSH, SW11 SW_PUSH, SW12 SW_PUSH, SW14 SW_PUSH, SW15 SW_PUSH, SW16 SW_PUSH, SW17 SW_PUSH, SW18 SW_PUSH, SW2 SW_PUSH, SW20 SW_PUSH, SW21 SW_PUSH, SW3 SW_PUSH, SW4 SW_PUSH, SW5 SW_PUSH, SW6 SW_PUSH, SW8 SW_PUSH, SW9 SW_PUSH, U1 ProMicro

Commit message: Update compact low
Parts:
- RSW1: footprint foostan:ResetSW -> * duckyb-collection:SMD_RST_SW [B3U-1000P(M)]
- turned RSW1 to -90 degrees
Routing:
- net reset: track 29.7 -> 34.9 mm, vias 0 -> 1
- net GND: track 381.5 -> 385.3 mm, vias 0 -> 1
- net Net-(U1-Pad12): track 35.4 -> 34.2 mm
- net col3: track 82.9 -> 83.9 mm
Other:
- net class Default removed
- board text added: "GND"
- board text added: "Pro-micro FACE DOWN"
- board text added: "Pro-micro FACE UP"
- board text added: "RAW"
- board text added: "RST"
- board text added: "VCC"
